File: wifi-floppy/hardware/wifi_floppy.kicad_sch (KiCad schematic)
At the start: 25 parts, among them J1 Conn_02x17_Odd_Even, J2 Conn_01x04, J3 Conn_01x04, J4 Conn_01x04, Q1 BSS138, Q2 BSS138, Q3 BSS138, Q4 BSS138, Q5 BSS138, Q6 BSS138, Q7 BSS138, Q8 BSS138, U1 RaspberryPi_Pico_W, U2 74LVC541A

Commit message: Add some pullup resistors to other inputs
Parts:
- added R1, R4, R5, R7, R8: 1k, wifi-floppy-lib:R_1206_3216Metric_Pad1.30x1.75mm_HandSolder, symbol wifi-floppy-lib:R_Small
- renumbered R6 to R10, R5 to R11, R1 to R2, R2 to R3, R3 to R6, R4 to R9
Connections:
- net +5V: now also R1.1, R4.1, R5.1, R7.1, R8.1
- net DIR_B: now also R5.2
- net SEL0_B: now also R8.2
- net SEL1_B: now also R7.2
- net SIDE_B: now also R1.2
- net STEP_B: now also R4.2
Other:
- moved on the sheet: D2, R6, R9

Commit message: Shutup two warning in schematics about power flags...
Other:
- moved on the sheet: C3, D1, J2
